File: hardware/easyeda/IchiPing-UNO-Q-Shields/uno_shield/ichiping_uno_q_shield.kicad_pcb (KiCad board)
At the start: 2 copper layers, 68.6 x 53.3 mm, 23 parts, among them J1 Power, J2 Digital/PWM, J3 Analog, J4 Digital/PWM

Commit message: Add 470uF filtering to 5V input
Parts:
- C_PWR_BULK: value 100u -> 470u 10V LOW ESR
Routing:
- net A5: track 77.8 -> 57.9 mm
- net GND: track 185.4 -> 194.5 mm
- net D13_SCK: track 47.1 -> 54.0 mm
- net D11_MOSI: track 57.8 -> 54.8 mm
- net D8_EXEC: track 29.0 -> 27.3 mm
- net D9_RAIN: track 43.0 -> 44.7 mm, vias 0 -> 1
- net +5V: track 57.8 -> 56.4 mm
- net +3V3: track 64.1 -> 64.7 mm
