File: hardware/easyeda/IchiPing-UNO-Q-Shields/audio_shield/ichiping_uno_q_audio_shield.kicad_pcb (KiCad board)
At the start: 2 copper layers, 46 x 53.3 mm, 12 parts, among them J14 UNO Breakout Carrier J14, J15 UNO Breakout Carrier J15

Commit message: Revise audio shield layout and schematic
Parts:
- removed SJ_MUTE: AMP SD mute, 
- added JP_MUTE: AMP SD MUTE (OPEN), , F.Cu at (55.0, 25.0)
- C1: value 10u -> 10u 10V
- moved J_MIC 57.1 mm to (61.0, 36.5)
- moved J_AMP_PWR 57.0 mm to (61.0, 23.5)
- moved J_AMP_SIG 57.0 mm to (61.0, 10.0)
- moved C2 22.4 mm to (54.0, 33.0)
- moved C3 22.1 mm to (54.0, 47.5)
- moved R_SD 20.7 mm to (49.0, 23.5)
- moved R_LR 19.4 mm to (48.0, 49.0)
- moved C1 19.0 mm to (48.0, 33.0)
- moved R_GAIN 15.1 mm to (44.0, 16.0)
Routing:
- net GND: track 110.0 -> 138.5 mm
- net AMP_SD: track 33.8 -> 13.2 mm, vias 2 -> 0
- net +1V8: track 46.6 -> 66.7 mm
- net +3V3: track 13.0 -> 30.2 mm
- net MIC_LR: track 15.6 -> 31.2 mm
- net MI2S0_WS: track 60.9 -> 76.5 mm
- net MI2S0_DATA0: track 29.9 -> 42.1 mm
- net +5V: track 52.9 -> 63.0 mm
- net AMP_GAIN: track 22.2 -> 27.5 mm
- net MI2S0_CLK: track 64.1 -> 66.2 mm, vias 0 -> 1
Other:
- board size 46 x 53.3 mm -> 79 x 53.3 mm
- board text added: "AMP PWR: SD GND VIN(5V)"
- board text added: "AMP SIG: LRC BCLK DIN GAIN"
- board text added: "I2S=1V8 ALL PARTS THT"
- board text added: "MIC: G 1V8 SD CK WS LR"
- board text added: "MUTE"
- board text added: "REV B 2026-08-25"
- board text removed: "AMP: LRC BCLK DIN GAIN"
- board text removed: "AMP: SD GND VIN(5V)"
- board text removed: "GAIN/LR=GND"
- board text removed: "I2S=1V8"
- board text removed: "MIC G 1V8 SD CK WS LR"
- board text removed: "REV A 2026-08-24"
