File: hardware/easyeda/IchiPing-UNO-Q-Shields/audio_shield/ichiping_uno_q_audio_shield.sch (KiCad schematic (older format))
At the start: 4 parts

Commit message: Revise audio shield layout and schematic
Parts:
- removed SJ_MUTE: XH2.54_VERTICAL_2, Connector_PinHeader_2.54mm:PinHeader_1x02_P2.54mm_Vertical, symbol Connector_Generic:Conn_01x02
- added C1: 10u 10V, Capacitor_THT:CP_Radial_D5.0mm_P2.00mm, symbol Device:C_Polarized
- added C2, C3: 100n, Capacitor_THT:C_Disc_D5.0mm_W2.5mm_P5.00mm, symbol Device:C
- added J14, J15: UNO Breakout Carrier, Connector_PinSocket_2.54mm:PinSocket_2x20_P2.54mm_Vertical, symbol Connector_Generic:Conn_02x20_Odd_Even
- added JP_MUTE: AMP SD MUTE (OPEN), Connector_PinHeader_2.54mm:PinHeader_1x02_P2.54mm_Vertical, symbol Connector_Generic:Conn_01x02
- added R_GAIN: 0R GAIN=GND, Resistor_THT:R_Axial_DIN0207_L6.3mm_D2.5mm_P10.16mm_Horizontal, symbol Device:R
- added R_LR: 0R MIC_LR=GND, Resistor_THT:R_Axial_DIN0207_L6.3mm_D2.5mm_P10.16mm_Horizontal, symbol Device:R
- added R_SD: 100k SD pull-up, Resistor_THT:R_Axial_DIN0207_L6.3mm_D2.5mm_P10.16mm_Horizontal, symbol Device:R
Connections:
- net labels added: +3V3
- wire segments 15 -> 42
- no-connect marks 0 -> 65
Other:
- note added: "Configuration and decoupling (THT)"
- note added: "IchiPing UNO Q Audio Shield - complete circuit"
- note added: "J14: 5/6=GND, 7/9=+5V, 13/15=+3V3, 19/21=+1V8"
- note added: "J15: 23/30/40=GND, 32=CLK, 34=WS, 36=DATA0(mic), 38=DATA1(amp)"
- note added: "JP_MUTE open: amplifier enabled by R_SD. Fit shunt: SD forced Low / mute."
- note added: "QRB2210 MI2S0 is 1.8 V logic. Confirm Device Tree and ALSA direction before fitting modules."
- note removed: "IchiPing UNO Q Audio Shield"
- note removed: "J15-32/34/36/38 = CLK/WS/DATA0/DATA1; J14 supplies +1V8 and +5V."
